File: vat_rev1/vat_rev1.kicad_sch (KiCad schematic)
At the start: 3 parts

Commit message: I think its mostly chilling
Parts:
- removed L1: L, symbol Device:L
- added C3, C5: 1uF, PCM_JLCPCB:C_1206, symbol Device:C
- added C4, C6: 0.1uF, PCM_JLCPCB:C_0603, symbol Device:C
- added D1: D_Schottky, symbol Device:D_Schottky
- added H1, H2, H3, H4: MountingHole_Pad, ssi_mountinghole:MountingHole_3.2mm_M3_DIN965_PadMOD, symbol Mechanical:MountingHole_Pad
- added J1: MAG_NOZZLE, Connector_AMASS:AMASS_XT60PW-F_1x02_P7.20mm_Horizontal, symbol Connector_Generic:Conn_01x02
- added JP1: Jumper_3_Open, PCM_SparkFun-Connector:ScrewTerminal_1x03_P3.5mm_Horizontal_Black, symbol Jumper:Jumper_3_Open
- added MAG_NOZZLE_INDUCTOR1: 50-60uH, symbol Device:L
- added Q1: IPB017N10N5ATMA1, Package_TO_SOT_SMD:TO-263-7_TabPin4, symbol Simulation_SPICE:NMOS
- added R1: 1m, symbol Device:R_US
- added R2, R3: 33K, symbol Device:R_US
- added R4, R5: 4.7, Resistor_SMD:R_0805_2012Metric, symbol Device:R_US
- added R6: 100k, symbol Device:R_US
- added TP1, TP2, TP3, TP4: TestPoint, TestPoint:TestPoint_Pad_1.5x1.5mm, symbol Connector:TestPoint
- added U1: 1EDN8550B, Package_TO_SOT_SMD:SOT-23-6, symbol Driver_FET:1EDN8550B
- C1: value C -> 470uF
- C2: value C -> 470uF; now not fitted
Connections:
- net GND: now also C1.2, C2.2, C3.2, C4.2, C5.2, C6.2, H1.1, H2.1, H3.1, H4.1, R1.1, R2.1, R6.1, U1.2 (GND)
- net VBUS: now also C5.1, C6.1, JP1.1 (A), U1.4 (VDD)
- net V_COIL: now reaches C1.1
- net V_COIL: now also C2.1, C3.1, C4.1, D1.1 (K), J1.1 (Pin_1), JP1.2 (C), TP3.1
- new net: R2.2, U1.1 (IN-)
- new net: R3.2, U1.3 (IN+)
- new net: R5.1, U1.5 (OUT_SRC)
- new net: R4.1, U1.6 (OUT_SNK)
- new net: Q1.3 (S), R1.2, R6.2
- new net: Q1.2 (G), R4.2, R5.2
- new net CL_SW: D1.2 (A), J1.2 (Pin_2), Q1.1 (D), TP4.1
- new net TRIG: R3.1
- new net V_BUS: TP2.1
- new net V_REG: JP1.3 (B), TP1.1
Other:
- note added: "33K for 3V3 Input"
- note added: "Conservative Values, can dec later"
- note added: "MAG_NOZZLE_CIRCUIT"
- note added: "MAX 22V so maybe VBUS?"
- note added: "MOUNTING HOLES"
- note added: "NEED FIND FP FOR THESE"
- note added: "PASSTHROUGH"
- note added: "POWER_SEL"
- note added: "PROTECTION"
- note added: "Regulation"
- note added: "SHUNT"
- note added: "TEST_POINTS"
- note removed: "BUCK and Such"
